File: 004_dzulov_zakon/004_dzulov_zakon.kicad_sch (KiCad schematic)
At the start: 8 parts, among them J2 Screw_Terminal_01x02

Commit message: julll.
Parts:
- added HS1: Heatsink, symbol Mechanical:Heatsink
- added J1, J3: Conn_01x01_Socket, Connector_PinSocket_2.54mm:PinSocket_1x01_P2.54mm_Vertical, symbol Connector:Conn_01x01_Socket
- added R2: 100k, Resistor_SMD:R_1206_3216Metric_Pad1.30x1.75mm_HandSolder, symbol Device:R
Connections:
- net 0: now also J3.1 (Pin_1), R2.2
- net Input voltage: now also J1.1 (Pin_1), R2.1
Other:
- note added: "otpornik okružen bakrom"
- note added: "zamneljivi i zapaljiv otpornik"
- title: Redna i paralelna otpornost -> Džulov zakon
- moved on the sheet: R1
