File: 004_dzulov_zakon/004_dzulov_zakon.kicad_pcb (KiCad board)
At the start: 2 copper layers, 45 x 45 mm, 12 parts, among them J2 Screw_Terminal_01x02, SW1 SW_Push, SW2 SW_Push

Commit message: julll.
Parts:
- removed C1, C2: 100u, Capacitor_THT:CP_Radial_D8.0mm_P3.50mm
- removed R6: 100k, Resistor_SMD:R_1206_3216Metric_Pad1.30x1.75mm_HandSolder
- removed REF**: ele_petnica_logo, PEP:ele_petnica_logo
- removed SW1, SW2: SW_Push, Button_Switch_THT:SW_PUSH_6mm_H4.3mm
- added J1: Conn_01x01_Socket, Connector_PinSocket_2.54mm:PinSocket_1x01_P2.54mm_Vertical, F.Cu at (142.0, 81.0)
- added J3: Conn_01x01_Socket, Connector_PinSocket_2.54mm:PinSocket_1x01_P2.54mm_Vertical, F.Cu at (142.0, 89.0)
- added R2: 100k, Resistor_SMD:R_1206_3216Metric_Pad1.30x1.75mm_HandSolder, F.Cu at (112.0, 84.0)
- added R3: 100k, Resistor_SMD:R_1206_3216Metric_Pad1.30x1.75mm_HandSolder, F.Cu at (125.0, 84.0)
- added R4: 100k, Resistor_SMD:R_1206_3216Metric_Pad1.30x1.75mm_HandSolder, F.Cu at (131.0, 84.0)
- moved R1 11.7 mm to (119.0, 84.0), turned to -90 degrees
Connections:
- R1 pad 1: Net-(R1-Pad1) -> Input voltage
- R1 pad 2: Output voltage -> 0
Routing:
- net Output voltage: track 14.2 -> 0.00 mm
- net Net-(R6-Pad1): track 9.66 -> 0.00 mm
- net Net-(R1-Pad1): track 9.66 -> 0.00 mm
- net Net-(C1-Pad2): track 6.00 -> 0.00 mm
- net Input voltage: track 39.2 -> 43.0 mm
Other:
- board text added: "Džulov zakon"
- board text added: "Light emiting resistor"
- board text added: "PEP 004"
- board text removed: "PEP 006"
- board text removed: "Punjenje / pražnjenje kondenzatora"
- board text removed: "prazni"

Commit message: Džul update.
Parts:
- moved J1 9.22 mm to (144.0, 90.0)
- moved J3 8.25 mm to (144.0, 81.0)
- moved R1 5.39 mm to (124.0, 86.0), turned to 90 degrees
- moved R3 5.39 mm to (130.0, 86.0), turned to 90 degrees
- moved R4 5.39 mm to (136.0, 86.0), turned to 90 degrees
- moved R2 2.24 mm to (113.0, 86.0), turned to 90 degrees
Routing:
- net Input voltage: track 43.0 -> 59.5 mm, vias 0 -> 4
- net 0: track 0.00 -> 7.35 mm, vias 109 -> 113
- added copper zone on F.Cu, net Input voltage
