File: PEP008_V1_strujno_naponska_karakteristika/PEP008_V1_strujno_naponska_karakteristika.kicad_pcb (KiCad board)
At the start: 2 copper layers, 45 x 45 mm, 16 parts, among them J2 Screw_Terminal_01x02, SW1 SW_Push, SW2 SW_Push

Commit message: PEP008 update.
Parts:
- removed 100uF: 100u, Capacitor_THT:CP_Radial_D8.0mm_P3.50mm
- added C1: 100uF, Capacitor_THT:C_Disc_D5.0mm_W2.5mm_P2.50mm, F.Cu at (127.8, 81.0)
Routing:
- net Net-(C1-Pad2): track 16.5 -> 17.1 mm
