File: PEP004-V1-matrica_otpornika/PEP004-V1-matrica_otpornika/PEP004-V1-matrica_otpornika.kicad_pcb (KiCad board)
At the start: 2 copper layers, 90 x 45 mm, 39 parts, among them J1 Screw_Terminal_01x02, SW1 SW_Push, SW10 SW_Push, SW11 SW_Push, SW12 SW_Push, SW13 SW_Push, SW14 SW_Push, SW15 SW_Push, SW16 SW_Push, SW2 SW_Push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

Commit message: PEP007 final update, ready for production.
Parts:
- removed D2: LED, LED_SMD:LED_1206_3216Metric_Pad1.42x1.75mm_HandSolder
- removed REF**: ele_petnica_logo, PEP_library:ele_petnica_logo
- removed REF** (x8): R_silk_symbol, PEP_library:R_silk_symbol
- added D1: LED, LED_SMD:LED_0603_1608Metric_Pad1.05x0.95mm_HandSolder, F.Cu at (185.0, 81.0)
- J1: footprint TerminalBlock_Phoenix:TerminalBlock_Phoenix_MKDS-1,5-2-5.08_1x02_P5.08mm_Horizontal -> PEP_library:TerminalBlock_Phoenix_MKDS-1,5-2-5.08_1x02_P5.08mm_Horizontal
- R1, R6: value 470 -> 1k; footprint Resistor_SMD:R_1206_3216Metric_Pad1.30x1.75mm_HandSolder -> PEP_library:R_smd
- R2: value 470 -> 2.2k; footprint Resistor_SMD:R_1206_3216Metric_Pad1.30x1.75mm_HandSolder -> PEP_library:R_smd
- R3: value 470 -> 22k; footprint Resistor_SMD:R_1206_3216Metric_Pad1.30x1.75mm_HandSolder -> PEP_library:R_smd
- R4: value 470 -> 10k; footprint Resistor_SMD:R_1206_3216Metric_Pad1.30x1.75mm_HandSolder -> PEP_library:R_smd
- R5: value 470 -> 220; footprint Resistor_SMD:R_1206_3216Metric_Pad1.30x1.75mm_HandSolder -> PEP_library:R_smd
- R7: value 470 -> 47k; footprint Resistor_SMD:R_1206_3216Metric_Pad1.30x1.75mm_HandSolder -> PEP_library:R_smd
- R8: value 470 -> 4.7k; footprint Resistor_SMD:R_1206_3216Metric_Pad1.30x1.75mm_HandSolder -> PEP_library:R_smd
- moved H4 207.0 mm to (3.02, 10.1)
- moved H3 196.3 mm to (3.02, 3.02)
- moved SW14 0.86 mm to (175.0, 76.7)
- moved SW15 0.86 mm to (175.0, 85.3)
- moved SW6 0.86 mm to (153.8, 76.7)
- moved SW7 0.86 mm to (153.8, 85.3)
- moved SW10 0.86 mm to (164.4, 76.7)
- moved SW11 0.86 mm to (164.4, 85.3)
- moved SW2 0.86 mm to (143.2, 76.7)
- moved SW3 0.86 mm to (143.2, 85.3)
- moved SW1 0.84 mm to (143.1, 68.0)
- moved SW13 0.84 mm to (175.0, 68.0)
- moved SW5 0.84 mm to (153.8, 68.0)
- moved SW9 0.84 mm to (164.4, 68.0)
- moved SW12 0.84 mm to (164.4, 94.0)
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Connections:
- R2 pad 2: Net-(R5-Pad2) -> Net-(R2-Pad2)
- SW10 pad 1: Net-(R5-Pad2) -> Net-(R2-Pad2)
- SW14 pad 1: Net-(R5-Pad2) -> Net-(R2-Pad2)
- SW2 pad 1: Net-(R5-Pad2) -> Net-(R2-Pad2)
- SW6 pad 1: Net-(R5-Pad2) -> Net-(R2-Pad2)
Routing:
- net 0: track 0.00 -> 94.8 mm, vias 170 -> 171
- net Net-(R2-Pad2): track 0.00 -> 45.5 mm
- net Net-(R5-Pad2): track 82.2 -> 57.8 mm
- net Net-(R8-Pad2): track 36.7 -> 58.1 mm
- net Net-(R6-Pad2): track 36.3 -> 57.6 mm
- net Net-(R7-Pad2): track 36.9 -> 58.1 mm
- net 9V: track 45.2 -> 43.5 mm
- net Net-(D1-A): track 63.1 -> 64.2 mm
Other:
- board text removed: "+"
- board text removed: "-"
