File: PEP004-V1-matrica_otpornika/PEP004-V1-matrica_otpornika/PEP004-V1-matrica_otpornika.kicad_sch (KiCad schematic)
At the start: 30 parts, among them J1 Screw_Terminal_01x02, SW1 SW_Push, SW10 SW_Push, SW11 SW_Push, SW12 SW_Push, SW13 SW_Push, SW14 SW_Push, SW15 SW_Push, SW16 SW_Push, SW2 SW_Push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

Commit message: PEP007 final update, ready for production.
Parts:
- removed D2: LED, LED_SMD:LED_1206_3216Metric_Pad1.42x1.75mm_HandSolder, symbol Device:LED
- added D1: LED, LED_SMD:LED_0603_1608Metric_Pad1.05x0.95mm_HandSolder, symbol Device:LED
- J1: footprint TerminalBlock_Phoenix:TerminalBlock_Phoenix_MKDS-1,5-2-5.08_1x02_P5.08mm_Horizontal -> PEP_library:TerminalBlock_Phoenix_MKDS-1,5-2-5.08_1x02_P5.08mm_Horizontal
- R1, R2, R3, R4, R5, R7, R8: footprint Resistor_SMD:R_1206_3216Metric_Pad1.30x1.75mm_HandSolder -> PEP_library:R_smd
- R6: value 100k -> 1k; footprint Resistor_SMD:R_1206_3216Metric_Pad1.30x1.75mm_HandSolder -> PEP_library:R_smd
Connections:
- net 0: now also D1.1 (K)
- net at R5.1, R6.1, R7.1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: now also D1.2 (A)
Changed lines of the file:
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@@
 	(wire
 		(pts
-			(xy 154.94 35.56) (xy 154.94 43.18)
-		)
-		(stroke
-			(width 0)
-			(type default)
-		)
-	)
-	(wire
-		(pts
-			(xy 187.96 39.37) (xy 191.77 39.37)
+			(xy 154.94 36.83) (xy 154.94 43.18)
 		)
 		(stroke
@@
 	(wire
 		(pts
-			(xy 242.57 43.18) (xy 242.57 31.75)
+			(xy 242.57 43.18) (xy 242.57 33.02)
 		)
 		(stroke
@@
 	(wire
 		(pts
-			(xy 218.44 43.18) (xy 218.44 35.56)
+			(xy 218.44 43.18) (xy 218.44 36.83)
 		)
 		(stroke
@@
 	(wire
 		(pts
-			(xy 242.57 31.75) (xy 149.86 31.75)
+			(xy 242.57 33.02) (xy 149.86 33.02)
 		)
 		(stroke
@@
 	(wire
 		(pts
-			(xy 218.44 35.56) (xy 154.94 35.56)
+			(xy 218.44 36.83) (xy 154.94 36.83)
 		)
 		(stroke
@@
 	(wire
 		(pts
-			(xy 158.75 38.1) (xy 187.96 38.1)
+			(xy 158.75 39.37) (xy 191.77 39.37)
 		)
 		(stroke
@@
 	(wire
 		(pts
-			(xy 149.86 31.75) (xy 149.86 43.18)
+			(xy 149.86 33.02) (xy 149.86 43.18)
 		)
 		(stroke
@@
 	(wire
 		(pts
-			(xy 158.75 43.18) (xy 158.75 38.1)
+			(xy 158.75 43.18) (xy 158.75 39.37)
 		)
 		(stroke
@@
 		(pts
 			(xy 154.94 62.23) (xy 154.94 68.58)
-		)
-		(stroke
-			(width 0)
-			(type default)
-		)
-	)
-	(wire
-		(pts
-			(xy 187.96 38.1) (xy 187.96 39.37)
 		)
 		(stroke
@@
 			(width 0)
 			(type default)
-			(color 110 183 49 1)
 		)
 		(fill
@@
 			(width 0)
 			(type default)
-			(color 110 183 49 1)
 		)
 		(fill
@@
 			(width 0)
 			(type default)
-			(color 110 183 49 1)
 		)
 		(fill
@@
 			(font
 				(size 2.54 2.54)
-				(color 110 183 49 1)
 			)
 			(justify left bottom)
@@
 			(font
 				(size 2.54 2.54)
-				(color 110 183 49 1)
 			)
 		)
@@
 			(font
 				(size 2.54 2.54)
-				(color 110 183 49 1)
 			)
 			(justify left bottom)
@@
 	)
 	(symbol
+		(lib_id "Device:LED")
+		(at 214.63 114.3 90)
+		(unit 1)
+		(exclude_from_sim no)
+		(in_bom yes)
+		(on_board yes)
+		(dnp no)
+		(fields_autoplaced yes)
+		(property "Reference" "D1"
+			(at 218.44 114.6175 90)
+			(effects
+				(font
+					(size 1.27 1.27)
+				)
+				(justify right)
+			)
+		)
+		(property "Value" "LED"
+			(at 218.44 117.1575 90)
+			(effects
+				(font
+					(size 1.27 1.27)
+				)
+				(justify right)
+			)
+		)
+		(property "Footprint" "LED_SMD:LED_0603_1608Metric_Pad1.05x0.95mm_HandSolder"
+			(at 214.63 114.3 0)
+			(effects
+				(font
+					(size 1.27 1.27)
+				)
+				(hide yes)
+			)
+		)
+		(property "Datasheet" "~"
+			(at 214.63 114.3 0)
+			(effects
+				(font
+					(size 1.27 1.27)
+				)
+				(hide yes)
+			)
+		)
+		(property "Description" ""
+			(at 214.63 114.3 0)
+			(effects
+				(font
+					(size 1.27 1.27)
+				)
+				(hide yes)
+			)
+		)
+		(pin "1"
+		)
+		(pin "2"
+		)
+		(instances
+			(project "PEP004-V1-matrica_otpornika"
+				(path "/4bec5ddf-adbf-41fb-a069-c7630bb0044a"
+					(reference "D1")
+					(unit 1)
+				)
+			)
+		)
+	)
+	(symbol
 		(lib_id "Switch:SW_Push")
 		(at 196.85 68.58 0)
@@
 	)
 	(symbol
-		(lib_id "Device:LED")
-		(at 214.63 114.3 90)
-		(unit 1)
-		(exclude_from_sim no)
-		(in_bom yes)
-		(on_board yes)
-		(dnp no)
-		(fields_autoplaced yes)
-		(property "Reference" "D2"
-			(at 218.44 114.6175 90)
-			(effects
-				(font
-					(size 1.27 1.27)
-				)
-				(justify right)
-			)
-		)
-		(property "Value" "LED"
-			(at 218.44 117.1575 90)
-			(effects
-				(font
-					(size 1.27 1.27)
-				)
-				(justify right)
-			)
-		)
-		(property "Footprint" "LED_SMD:LED_1206_3216Metric_Pad1.42x1.75mm_HandSolder"
-			(at 214.63 114.3 0)
-			(effects
-				(font
-					(size 1.27 1.27)
-				)
-				(hide yes)
-			)
-		)
-		(property "Datasheet" "~"
-			(at 214.63 114.3 0)
-			(effects
-				(font
-					(size 1.27 1.27)
-				)
-				(hide yes)
-			)
-		)
-		(property "Description" ""
-			(at 214.63 114.3 0)
-			(effects
-				(font
-					(size 1.27 1.27)
-				)
-				(hide yes)
-			)
-		)
-		(pin "1"
-		)
-		(pin "2"
-		)
-		(instances
-			(project "sa matricom"
-				(path "/4bec5ddf-adbf-41fb-a069-c7630bb0044a"
-					(reference "D2")
-					(unit 1)
-				)
-			)
-		)
-	)
-	(symbol
 		(lib_id "Switch:SW_Push")
 		(at 172.72 43.18 0)
@@
 			)
 		)
-		(property "Footprint" "Resistor_SMD:R_1206_3216Metric_Pad1.30x1.75mm_HandSolder"
+		(property "Footprint" "PEP_library:R_smd"
 			(at 142.24 44.958 90)
 			(effects
@@
 			)
 		)
-		(property "Footprint" "Resistor_SMD:R_1206_3216Metric_Pad1.30x1.75mm_HandSolder"
+		(property "Footprint" "PEP_library:R_smd"
 			(at 254.508 93.98 90)
 			(effects
@@
 			)
 		)
-		(property "Footprint" "Resistor_SMD:R_1206_3216Metric_Pad1.30x1.75mm_HandSolder"
+		(property "Footprint" "PEP_library:R_smd"
 			(at 179.578 93.98 90)
 			(effects
@@
 			)
 		)
-		(property "Footprint" "Resistor_SMD:R_1206_3216Metric_Pad1.30x1.75mm_HandSolder"
+		(property "Footprint" "PEP_library:R_smd"
 			(at 230.378 93.98 90)
 			(effects
@@
 			)
 		)
-		(property "Footprint" "Resistor_SMD:R_1206_3216Metric_Pad1.30x1.75mm_HandSolder"
+		(property "Footprint" "PEP_library:R_smd"
 			(at 142.24 57.658 90)
 			(effects
@@
 				(font
 					(size 1.27 1.27)
+					(thickness 0.254)
+					(bold yes)
 				)
 				(hide yes)
@@
 			)
 		)
-		(property "Footprint" "Resistor_SMD:R_1206_3216Metric_Pad1.30x1.75mm_HandSolder"
+		(property "Footprint" "PEP_library:R_smd"
 			(at 142.24 70.358 90)
 			(effects
@@
 			)
 		)
-		(property "Footprint" "TerminalBlock_Phoenix:TerminalBlock_Phoenix_MKDS-1,5-2-5.08_1x02_P5.08mm_Horizontal"
+		(property "Footprint" "PEP_library:TerminalBlock_Phoenix_MKDS-1,5-2-5.08_1x02_P5.08mm_Horizontal"
 			(at 58.42 60.96 0)
 			(effects
@@
 			)
 		)
-		(property "Footprint" "Resistor_SMD:R_1206_3216Metric_Pad1.30x1.75mm_HandSolder"
+		(property "Footprint" "PEP_library:R_smd"
 			(at 142.24 83.058 90)
 			(effects
@@
 		(fields_autoplaced yes)
 		(property "Reference" "R6"
-			(at 195.58 93.98 90)
-			(effects
-				(font
-					(size 1.27 1.27)
-				)
-			)
-		)
-		(property "Value" "100k"
-			(at 198.12 93.98 90)
-			(effects
-				(font
-					(size 1.27 1.27)
-				)
-			)
-		)
-		(property "Footprint" "Resistor_SMD:R_1206_3216Metric_Pad1.30x1.75mm_HandSolder"
+			(at 204.47 92.7099 0)
+			(effects
+				(font
+					(size 1.27 1.27)
+				)
+				(justify right)
+			)
+		)
+		(property "Value" "1k"
+			(at 204.47 95.2499 0)
+			(effects
+				(font
+					(size 1.27 1.27)
+				)
+				(justify right)
+			)
+		)
+		(property "Footprint" "PEP_library:R_smd"
 			(at 203.708 93.98 90)
 			(effects
