File: PEP001-V1-naponski_razdelnik/PEP001-V1-naponski_razdelnik.kicad_sch (KiCad schematic)
At the start: 11 parts, among them J1 Screw_Terminal_01x02

Commit message: PEP001 - Only LCSL linking left.
Parts:
- R2, R4: value 90k -> 81k
Changed lines of the file:
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@@
 		(fields_autoplaced yes)
 		(property "Reference" "R2"
-			(at 152.4 34.29 0)
-			(effects
-				(font
-					(size 1.27 1.27)
-				)
-				(justify left)
-			)
-		)
-		(property "Value" "90k"
-			(at 152.4 36.83 0)
+			(at 152.4 34.2899 0)
+			(effects
+				(font
+					(size 1.27 1.27)
+				)
+				(justify left)
+			)
+		)
+		(property "Value" "81k"
+			(at 152.4 36.8299 0)
 			(effects
 				(font
@@
 		(fields_autoplaced yes)
 		(property "Reference" "R4"
-			(at 93.98 33.02 0)
+			(at 93.98 33.0199 0)
 			(effects
 				(font
@@
 			)
 		)
-		(property "Value" "90k"
-			(at 93.98 35.56 0)
-			(effects
-				(font
+		(property "Value" "81k"
+			(at 93.98 35.5599 0)
+			(effects
+				(font
