File: PEP001-V1-naponski_razdelnik/PEP001-V1-naponski_razdelnik.kicad_sch (KiCad schematic)
At the start: 11 parts, among them J1 Screw_Terminal_01x02

Commit message: Update 1,2,3,4,5,7, lib.
Parts:
- removed J1: Screw_Terminal_01x02, TerminalBlock_Phoenix:TerminalBlock_Phoenix_MKDS-1,5-2-5.08_1x02_P5.08mm_Horizontal, symbol Connector:Screw_Terminal_01x02
- removed R1: 10k, Resistor_SMD:R_1206_3216Metric_Pad1.30x1.75mm_HandSolder, symbol Device:R
- removed R2: 82k, Resistor_SMD:R_1206_3216Metric_Pad1.30x1.75mm_HandSolder, symbol Device:R
- removed R3: 10k, Resistor_THT:R_Axial_DIN0207_L6.3mm_D2.5mm_P15.24mm_Horizontal, symbol Device:R
- removed R4: 82k, Resistor_THT:R_Axial_DIN0207_L6.3mm_D2.5mm_P15.24mm_Horizontal, symbol Device:R
- added J1: Klema, PEP_library:TerminalBlock_Phoenix_MKDS-1,5-2-5.08_1x02_P5.08mm_Horizontal, symbol PEP_library:Klema
- added R1: 10k, PEP_library:R_smd_1206, symbol PEP_library:R_SMD
- added R2: 82k, PEP_library:R_smd_1206, symbol PEP_library:R_SMD
- added R3: 10k, PEP_library:R_Axial_DIN0207_L6.3mm_D2.5mm_P15.24mm_Horizontal, symbol PEP_library:R_THT
- added R4: 82k, PEP_library:R_Axial_DIN0207_L6.3mm_D2.5mm_P15.24mm_Horizontal, symbol PEP_library:R_THT
Connections:
- net 0: now also J1.2 (Pin_2), R1.2, R3.2
- net 9V: now also J1.1 (Pin_1), R2.1, R4.1
- net at TP2.1: now also R1.1, R2.2
- net at TP1.1: now also R3.1, R4.2
