File: PEP002-V1-strujni_razdelnik/PEP002-V1-strujni_razdelnik.kicad_pcb (KiCad board)
At the start: 2 copper layers, 45 x 45 mm, 21 parts, among them J1 Screw_Terminal_01x02

Commit message: PEP002 - Only LCSC linking left.
Parts:
- added REF**: ele_petnica_logo, PEP_library:ele_petnica_logo, F.Cu at (116.0, 69.5)
- R2, R4: value 90k -> 81k
- moved TP6 0.50 mm to (133.0, 81.0)
- moved TP8 0.50 mm to (138.5, 81.0)
Routing:
- net 0: track 3.90 -> 50.0 mm, vias 111 -> 0
- net (no net): vias 0 -> 109
- removed copper zone on B.Cu, net 0
- removed copper zone on F.Cu, net 0
