File: PEP002-V1-strujni_razdelnik/PEP002-V1-strujni_razdelnik.kicad_sch (KiCad schematic)
At the start: 21 parts, among them J1 Screw_Terminal_01x02

Commit message: PEP002 - Only LCSC linking left.
Parts:
- R2, R4: value 90k -> 81k
Changed lines of the file:
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@@
 		(fields_autoplaced yes)
 		(property "Reference" "R2"
-			(at 154.94 52.07 0)
+			(at 154.94 52.0699 0)
 			(effects
 				(font
@@
 			)
 		)
-		(property "Value" "90k"
-			(at 154.94 54.61 0)
+		(property "Value" "81k"
+			(at 154.94 54.6099 0)
 			(effects
 				(font
@@
 				)
 				(justify left)
+				(hide yes)
 			)
 		)
@@
 		(fields_autoplaced yes)
 		(property "Reference" "R4"
-			(at 91.44 49.53 0)
+			(at 91.44 49.5299 0)
 			(effects
 				(font
@@
 			)
 		)
-		(property "Value" "90k"
-			(at 91.44 52.07 0)
-			(effects
-				(font
+		(property "Value" "81k"
+			(at 91.44 52.0699 0)
+			(effects
+				(font
