File: PEP002-V1-strujni_razdelnik/PEP002-V1-strujni_razdelnik.kicad_sch (KiCad schematic)
At the start: 21 parts, among them J1 Screw_Terminal_01x02

Commit message: Update 1,2,3,4,5,7, lib.
Parts:
- J1: footprint TerminalBlock_Phoenix:TerminalBlock_Phoenix_MKDS-1,5-2-5.08_1x02_P5.08mm_Horizontal -> PEP_library:TerminalBlock_Phoenix_MKDS-1,5-2-5.08_1x02_P5.08mm_Horizontal
- renumbered JP4 to JP1, JP3 to JP2, JP2 to JP3, JP1 to JP4, R4 to R1, R3 to R2, R2 to R3, R1 to R4, TP2 to TP1, TP3 to TP2, TP5 to TP3, TP7 to TP4, TP1 to TP5, TP4 to TP6, TP6 to TP7
Changed lines of the file:
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@@
 		(dnp no)
 		(fields_autoplaced yes)
-		(property "Reference" "TP4"
+		(property "Reference" "TP6"
 			(at 105.918 38.1 90)
 			(effects
@@
 			(project "002_strujni_razdelnik"
 				(path "/4bec5ddf-adbf-41fb-a069-c7630bb0044a"
-					(reference "TP4")
+					(reference "TP6")
 					(unit 1)
 				)
@@
 		(dnp no)
 		(fields_autoplaced yes)
-		(property "Reference" "R2"
+		(property "Reference" "R3"
 			(at 154.94 52.0699 0)
 			(effects
@@
 			(project "002_strujni_razdelnik"
 				(path "/4bec5ddf-adbf-41fb-a069-c7630bb0044a"
-					(reference "R2")
+					(reference "R3")
 					(unit 1)
 				)
@@
 		(dnp no)
 		(fields_autoplaced yes)
-		(property "Reference" "TP3"
+		(property "Reference" "TP2"
 			(at 105.918 22.86 90)
 			(effects
@@
 			(project "002_strujni_razdelnik"
 				(path "/4bec5ddf-adbf-41fb-a069-c7630bb0044a"
-					(reference "TP3")
+					(reference "TP2")
 					(unit 1)
 				)
@@
 		(dnp no)
 		(fields_autoplaced yes)
-		(property "Reference" "R3"
+		(property "Reference" "R2"
 			(at 119.38 49.53 0)
 			(effects
@@
 			(project "002_strujni_razdelnik"
 				(path "/4bec5ddf-adbf-41fb-a069-c7630bb0044a"
-					(reference "R3")
+					(reference "R2")
 					(unit 1)
 				)
@@
 			)
 		)
-		(property "Footprint" "TerminalBlock_Phoenix:TerminalBlock_Phoenix_MKDS-1,5-2-5.08_1x02_P5.08mm_Horizontal"
+		(property "Footprint" "PEP_library:TerminalBlock_Phoenix_MKDS-1,5-2-5.08_1x02_P5.08mm_Horizontal"
 			(at 40.64 38.1 0)
 			(effects
@@
 					(size 1.27 1.27)
 				)
-				(hide yes)
 			)
 		)
@@
 		(dnp no)
 		(fields_autoplaced yes)
-		(property "Reference" "JP3"
+		(property "Reference" "JP2"
 			(at 115.57 36.83 90)
 			(effects
@@
 			(project "002_strujni_razdelnik"
 				(path "/4bec5ddf-adbf-41fb-a069-c7630bb0044a"
-					(reference "JP3")
+					(reference "JP2")
 					(unit 1)
 				)
@@
 		(dnp no)
 		(fields_autoplaced yes)
-		(property "Reference" "TP5"
+		(property "Reference" "TP3"
 			(at 141.478 25.4 90)
 			(effects
@@
 			(project "002_strujni_razdelnik"
 				(path "/4bec5ddf-adbf-41fb-a069-c7630bb0044a"
-					(reference "TP5")
+					(reference "TP3")
 					(unit 1)
 				)
@@
 		(dnp no)
 		(fields_autoplaced yes)
-		(property "Reference" "JP2"
+		(property "Reference" "JP3"
 			(at 151.13 36.83 90)
 			(effects
@@
 			(project "002_strujni_razdelnik"
 				(path "/4bec5ddf-adbf-41fb-a069-c7630bb0044a"
-					(reference "JP2")
+					(reference "JP3")
 					(unit 1)
 				)
@@
 		(dnp no)
 		(fields_autoplaced yes)
-		(property "Reference" "TP1"
+		(property "Reference" "TP5"
 			(at 77.978 38.1 90)
 			(effects
@@
 			(project "002_strujni_razdelnik"
 				(path "/4bec5ddf-adbf-41fb-a069-c7630bb0044a"
-					(reference "TP1")
+					(reference "TP5")
 					(unit 1)
 				)
@@
 		(dnp no)
 		(fields_autoplaced yes)
-		(property "Reference" "JP1"
+		(property "Reference" "JP4"
 			(at 179.07 36.83 90)
 			(effects
@@
 			(project "002_strujni_razdelnik"
 				(path "/4bec5ddf-adbf-41fb-a069-c7630bb0044a"
-					(reference "JP1")
+					(reference "JP4")
 					(unit 1)
 				)
@@
 		(on_board yes)
 		(dnp no)
-		(property "Reference" "R1"
+		(property "Reference" "R4"
 			(at 182.88 52.07 0)
 			(effects
@@
 			(project "002_strujni_razdelnik"
 				(path "/4bec5ddf-adbf-41fb-a069-c7630bb0044a"
-					(reference "R1")
+					(reference "R4")
 					(unit 1)
 				)
@@
 		(dnp no)
 		(fields_autoplaced yes)
-		(property "Reference" "TP7"
+		(property "Reference" "TP4"
 			(at 169.418 25.4 90)
 			(effects
@@
 			(project "002_strujni_razdelnik"
 				(path "/4bec5ddf-adbf-41fb-a069-c7630bb0044a"
-					(reference "TP7")
+					(reference "TP4")
 					(unit 1)
 				)
@@
 		(dnp no)
 		(fields_autoplaced yes)
-		(property "Reference" "JP4"
+		(property "Reference" "JP1"
 			(at 87.63 36.83 90)
 			(effects
@@
 			(project "002_strujni_razdelnik"
 				(path "/4bec5ddf-adbf-41fb-a069-c7630bb0044a"
-					(reference "JP4")
+					(reference "JP1")
 					(unit 1)
 				)
@@
 		(dnp no)
 		(fields_autoplaced yes)
-		(property "Reference" "TP6"
+		(property "Reference" "TP7"
 			(at 141.478 40.64 90)
 			(effects
@@
 			(project "002_strujni_razdelnik"
 				(path "/4bec5ddf-adbf-41fb-a069-c7630bb0044a"
-					(reference "TP6")
+					(reference "TP7")
 					(unit 1)
 				)
@@
 		(dnp no)
 		(fields_autoplaced yes)
-		(property "Reference" "R4"
+		(property "Reference" "R1"
 			(at 91.44 49.5299 0)
 			(effects
@@
 			(project "002_strujni_razdelnik"
 				(path "/4bec5ddf-adbf-41fb-a069-c7630bb0044a"
-					(reference "R4")
+					(reference "R1")
 					(unit 1)
 				)
@@
 		(dnp no)
 		(fields_autoplaced yes)
-		(property "Reference" "TP2"
+		(property "Reference" "TP1"
 			(at 77.978 22.86 90)
 			(effects
@@
 			(project "002_strujni_razdelnik"
 				(path "/4bec5ddf-adbf-41fb-a069-c7630bb0044a"
-					(reference "TP2")
-					(unit 1)
-				)
+					(reference "TP1")
+					(unit 1)
+				)
