File: PEP003-V1-redna_i_paralelna_otpornost/PEP003-V1-redna_i_paralelna_otpornost.kicad_pcb (KiCad board)
At the start: 2 copper layers, 90 x 45 mm, 41 parts, among them J1 Screw_Terminal_01x02

Commit message: PEP003_update
Routing:
- net 0: track 0.00 -> 73.7 mm
- net Net-(D1-A): track 41.4 -> 30.1 mm
- net 9V: track 127.7 -> 119.1 mm
Changed lines of the file:
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@@
 	)
 	(gr_line
-		(start 170 146)
-		(end 119.5 146)
+		(start 169.9 143.8)
+		(end 115.5 143.8)
 		(stroke
 			(width 0.15)
@@
 	)
 	(gr_line
-		(start 171 112.5375)
-		(end 171 109)
-		(stroke
-			(width 0.15)
-			(type default)
-		)
-		(layer "B.SilkS")
-	)
-	(gr_line
-		(start 115.5 144.5)
+		(start 115.5 143.8)
 		(end 115.5 121.5)
 		(stroke
@@
 	)
 	(gr_line
-		(start 175.5625 112.56875)
+		(start 175.5 112.7875)
 		(end 175.5 112.7875)
 		(stroke
@@
 	)
 	(gr_line
-		(start 162 109)
+		(start 162 112.725)
 		(end 162 128)
 		(stroke
@@
 	)
 	(gr_line
-		(start 166.4375 112.50625)
-		(end 175.5625 112.56875)
+		(start 166.375 112.725)
+		(end 175.5 112.7)
 		(stroke
 			(width 0.15)
@@
 	)
 	(gr_line
-		(start 166.4375 112.50625)
+		(start 166.375 112.725)
 		(end 166.375 112.725)
 		(stroke
@@
 	)
 	(gr_line
-		(start 116.5 146)
-		(end 115.5 144.5)
-		(stroke
-			(width 0.15)
-			(type default)
-		)
-		(layer "B.SilkS")
-	)
-	(gr_line
 		(start 148.823982 127.99638)
 		(end 147.423982 129.09638)
@@
 	)
 	(gr_line
-		(start 170 146)
-		(end 171 145.2875)
-		(stroke
-			(width 0.15)
-			(type default)
-		)
-		(layer "B.SilkS")
-	)
-	(gr_line
 		(start 159 126.89638)
 		(end 157.6 127.99638)
@@
 	)
 	(gr_line
-		(start 171 143.7875)
-		(end 171 145.2875)
-		(stroke
-			(width 0.15)
-			(type default)
-		)
-		(layer "B.SilkS")
-	)
-	(gr_line
-		(start 119.5 146)
-		(end 116.5 146)
-		(stroke
-			(width 0.15)
-			(type default)
-		)
-		(layer "B.SilkS")
-	)
-	(gr_line
 		(start 175.504223 114.2875)
-		(end 175.5 112.7875)
+		(end 175.5 112.7)
 		(stroke
 			(width 0.15)
@@
 	)
 	(gr_line
-		(start 171 109)
-		(end 162 109)
+		(start 166.5 112.725)
+		(end 162 112.725)
 		(stroke
 			(width 0.15)
@@
 	)
 	(segment
-		(start 117.5 144)
-		(end 115.5 142)
-		(width 1)
-		(layer "F.Cu")
-		(net 2)
-	)
-	(segment
-		(start 169.5 144)
-		(end 117.5 144)
-		(width 1)
-		(layer "F.Cu")
-		(net 2)
+		(start 106.3 126.38)
+		(end 106.3 121.6)
+		(width 1)
+		(layer "F.Cu")
+		(net 1)
+	)
+	(segment
+		(start 145.6 112.6)
+		(end 151.5 118.5)
+		(width 1)
+		(layer "F.Cu")
+		(net 1)
+	)
+	(segment
+		(start 151.5 127.8)
+		(end 151.7 128)
+		(width 1)
+		(layer "F.Cu")
+		(net 1)
+	)
+	(segment
+		(start 151.5 118.5)
+		(end 151.5 127.8)
+		(width 1)
+		(layer "F.Cu")
+		(net 1)
+	)
+	(segment
+		(start 106.3 121.6)
+		(end 115.3 112.6)
+		(width 1)
+		(layer "F.Cu")
+		(net 1)
+	)
+	(segment
+		(start 109 129.08)
+		(end 106.3 126.38)
+		(width 1)
+		(layer "F.Cu")
+		(net 1)
+	)
+	(segment
+		(start 151.5 128)
+		(end 151.7 128)
+		(width 1)
+		(layer "F.Cu")
+		(net 1)
+	)
+	(segment
+		(start 151.7 128)
+		(end 155.625 128)
+		(width 1)
+		(layer "F.Cu")
+		(net 1)
+	)
+	(segment
+		(start 115.3 112.6)
+		(end 145.6 112.6)
+		(width 1)
+		(layer "F.Cu")
+		(net 1)
 	)
 	(segment
@@
 	)
 	(segment
-		(start 115.5 142)
-		(end 115.5 125.5)
-		(width 1)
-		(layer "F.Cu")
-		(net 2)
-	)
-	(segment
 		(start 128.225 130.5)
 		(end 128.225 125.5)
@@
 	)
 	(segment
+		(start 164.9 141.7)
+		(end 124.5 141.7)
+		(width 1)
+		(layer "F.Cu")
+		(net 2)
+	)
+	(segment
+		(start 166.2625 140.3375)
+		(end 164.9 141.7)
+		(width 1)
+		(layer "F.Cu")
+		(net 2)
+	)
+	(segment
 		(start 114 124)
 		(end 109 124)
@@
 	)
 	(segment
-		(start 171 140.3375)
-		(end 171 142.5)
-		(width 1)
-		(layer "F.Cu")
-		(net 2)
-	)
-	(segment
 		(start 128.46 138.5)
 		(end 128.46 130.735)
@@
 	)
 	(segment
+		(start 171 140.3375)
+		(end 166.2625 140.3375)
+		(width 1)
+		(layer "F.Cu")
+		(net 2)
+	)
+	(segment
 		(start 128.225 125.5)
+		(end 115.5 125.5)
+		(width 1)
+		(layer "F.Cu")
+		(net 2)
+	)
+	(segment
+		(start 115.5 132.7)
 		(end 115.5 125.5)
 		(width 1)
@@
 	)
 	(segment
+		(start 124.5 141.7)
+		(end 115.5 132.7)
+		(width 1)
+		(layer "F.Cu")
+		(net 2)
+	)
+	(segment
 		(start 128.225 122)
 		(end 128.225 115.765)
@@
 	)
 	(segment
-		(start 171 142.5)
-		(end 169.5 144)
-		(width 1)
-		(layer "F.Cu")
-		(net 2)
-	)
-	(segment
 		(start 166.5 140.3375)
 		(end 171 140.3375)
@@
 	)
 	(segment
-		(start 162.5 126.5)
-		(end 161 128)
-		(width 1)
-		(layer "F.Cu")
-		(net 3)
-	)
-	(segment
-		(start 171 112.5)
-		(end 170 111.5)
-		(width 1)
-		(layer "F.Cu")
-		(net 3)
-	)
-	(segment
-		(start 171 115.7375)
-		(end 171 112.5)
-		(width 1)
-		(layer "F.Cu")
-		(net 3)
-	)
-	(segment
-		(start 162.5 112.5)
-		(end 162.5 126.5)
-		(width 1)
-		(layer "F.Cu")
-		(net 3)
-	)
-	(segment
-		(start 161 128)
-		(end 157.375 128)
+		(start 165.7375 115.7375)
+		(end 157.375 124.1)
 		(width 1)
 		(layer "F.Cu")
@@
 	)
 	(segment
-		(start 170 111.5)
-		(end 163.5 111.5)
+		(start 157.375 124.1)
+		(end 157.375 128)
 		(width 1)
 		(layer "F.Cu")
@@
 	)
 	(segment
-		(start 163.5 111.5)
-		(end 162.5 112.5)
-		(width 1)
-		(layer "F.Cu")
+		(start 171 115.7375)
+		(end 165.7375 115.7375)
+		(width 1)
+		(layer "F.Cu")

Commit message: PEP003 final commit, ready for production.
Parts:
- removed the REF** at (131.5, 139.6)
- removed the REF** at (131.4, 131.6)
- removed the REF** at (131.5, 115.1)
- removed the REF** at (166.4, 134.1)
- removed the REF** at (175.5, 124.5)
- removed the REF** at (166.4, 126.6)
- removed the REF** at (175.5, 116.8)
- removed the REF** at (131.5, 123.6)
- removed the REF** at (175.5, 139.0)
- removed the REF** at (166.4, 119.3)
- removed the REF** at (175.5, 131.5)
- removed the REF** at (166.4, 112.6)
- removed the REF** at (133.3, 123.6)
- removed the REF** at (133.3, 139.6)
- removed the REF** at (133.3, 131.6)
- removed the REF** at (133.3, 115.1)
- added REF**: JP_silk_symbol, PEP_library:JP_silk_symbol, F.Cu at (135.3, 87.6)
- added REF**: JP_silk_symbol, PEP_library:JP_silk_symbol, F.Cu at (179.3, 72.8)
- added REF**: R_silk_symbol, PEP_library:R_silk_symbol, F.Cu at (137.1, 79.6)
- added REF**: R_silk_symbol, PEP_library:R_silk_symbol, F.Cu at (170.2, 90.1)
- added REF**: JP_silk_symbol, PEP_library:JP_silk_symbol, F.Cu at (179.3, 80.5)
- added REF**: JP_silk_symbol, PEP_library:JP_silk_symbol, F.Cu at (135.3, 71.1)
- added REF**: R_silk_symbol, PEP_library:R_silk_symbol, F.Cu at (170.2, 75.3)
- added REF**: R_silk_symbol, PEP_library:R_silk_symbol, F.Cu at (170.2, 68.6)
- added REF**: R_silk_symbol, PEP_library:R_silk_symbol, F.Cu at (170.2, 82.6)
- added REF**: JP_silk_symbol, PEP_library:JP_silk_symbol, F.Cu at (135.3, 95.6)
- added REF**: JP_silk_symbol, PEP_library:JP_silk_symbol, F.Cu at (179.3, 87.5)
- added REF**: R_silk_symbol, PEP_library:R_silk_symbol, F.Cu at (137.1, 87.6)
- added REF**: JP_silk_symbol, PEP_library:JP_silk_symbol, F.Cu at (135.3, 79.6)
- added REF**: JP_silk_symbol, PEP_library:JP_silk_symbol, F.Cu at (179.3, 95.0)
- added REF**: R_silk_symbol, PEP_library:R_silk_symbol, F.Cu at (137.1, 95.6)
- added REF**: R_silk_symbol, PEP_library:R_silk_symbol, F.Cu at (137.1, 71.1)
- moved H4 44.2 mm to (189.0, 101.0)
- moved H1 44.2 mm to (109.0, 101.0)
- moved H2 44.2 mm to (109.0, 66.0)
- moved H3 44.2 mm to (189.0, 66.0)
- moved D1 44.2 mm to (160.3, 84.0)
- moved D2 44.2 mm to (154.5, 84.0)
- moved G*** 44.2 mm to (157.3, 72.5)
- moved J1 44.2 mm to (112.8, 80.0)
- moved JP1 44.2 mm to (179.3, 96.3)
- moved JP2 44.2 mm to (179.3, 88.8)
- moved JP3 44.2 mm to (179.3, 81.3)
- moved JP4 44.2 mm to (179.3, 74.1)
- moved JP5 44.2 mm to (132.3, 94.5)
- moved JP6 44.2 mm to (132.1, 86.5)
- moved JP7 44.2 mm to (132.1, 78.0)
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Connections:
- D1 pad 2: Net-(D1-A) -> (no net)
- D2 pad 2: Net-(D2-A) -> (no net)
- JP1 pad 2: Net-(JP1-B) -> (no net)
- JP2 pad 1: Net-(JP1-B) -> (no net)
- JP2 pad 2: Net-(JP2-B) -> (no net)
- JP3 pad 1: Net-(JP2-B) -> (no net)
- JP3 pad 2: Net-(JP3-B) -> (no net)
- JP4 pad 1: Net-(JP3-B) -> (no net)
- JP4 pad 2: Net-(D1-A) -> (no net)
- JP5 pad 2: Net-(JP5-B) -> (no net)
- JP6 pad 2: Net-(JP6-B) -> (no net)
- JP7 pad 2: Net-(JP7-B) -> (no net)
- JP8 pad 2: Net-(JP8-B) -> (no net)
- R1 pad 2: Net-(JP1-B) -> (no net)
- R2 pad 1: Net-(JP1-B) -> (no net)
- R2 pad 2: Net-(JP2-B) -> (no net)
- R3 pad 1: Net-(JP2-B) -> (no net)
- R3 pad 2: Net-(JP3-B) -> (no net)
- R4 pad 1: Net-(JP3-B) -> (no net)
- R4 pad 2: Net-(D1-A) -> (no net)
- R5 pad 1: Net-(D2-A) -> (no net)
- R5 pad 2: Net-(JP5-B) -> (no net)
- R6 pad 1: Net-(JP6-B) -> (no net)
- R6 pad 2: Net-(D2-A) -> (no net)
- R7 pad 1: Net-(JP7-B) -> (no net)
- R7 pad 2: Net-(D2-A) -> (no net)
- R8 pad 1: Net-(D2-A) -> (no net)
- R8 pad 2: Net-(JP8-B) -> (no net)
Routing:
- net (no net): track 0.00 -> 162.4 mm, vias 170 -> 0
- net Net-(D2-A): track 30.2 -> 0.00 mm
- net Net-(D1-A): track 30.1 -> 0.00 mm
- net Net-(JP1-B): track 22.6 -> 0.00 mm
- net Net-(JP3-B): track 22.5 -> 0.00 mm
- net Net-(JP2-B): track 22.2 -> 0.00 mm
- net Net-(JP8-B): track 8.95 -> 0.00 mm
- net Net-(JP7-B): track 8.69 -> 0.00 mm
- net Net-(JP6-B): track 8.69 -> 0.00 mm
- net Net-(JP5-B): track 8.45 -> 0.00 mm
- net 0: vias 0 -> 170

Commit message: Update 1,2,3,4,5,7, lib.
Parts:
- removed the G*** at (157.3, 72.5)
- added G***: LOGO, PEP_library:petnica_logo, F.Cu at (162.7, 91.0)
- moved REF** 18.8 mm to (153.9, 91.0)
- moved REF** 5.46 mm to (139.1, 99.6)
- moved REF** 5.46 mm to (140.8, 99.6)
- moved REF** 4.48 mm to (139.0, 90.1)
- moved REF** 4.48 mm to (140.8, 90.1)
- moved REF** 4.47 mm to (139.0, 68.5)
- moved REF** 4.47 mm to (140.8, 68.5)
- moved REF** 3.91 mm to (140.8, 78.1)
- moved REF** 3.91 mm to (139.0, 78.1)
- moved REF** 2.35 mm to (177.0, 72.8)
- moved REF** 2.35 mm to (167.9, 90.1)
- moved REF** 2.35 mm to (177.0, 80.5)
- moved REF** 2.35 mm to (167.9, 75.3)
- moved REF** 2.35 mm to (167.9, 68.6)
- moved REF** 2.35 mm to (167.9, 82.6)
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Other:
- board text added: "D1"
- board text added: "D2"
- board text added: "JP1"
- board text added: "JP2"
- board text added: "JP3"
- board text added: "JP4"
- board text added: "JP5"
- board text added: "JP6"
- board text added: "JP7"
- board text added: "JP8"
- board text added: "R1"
- board text added: "R2"
- board text added: "R3"
- board text added: "R4"
- board text added: "R5"
- board text added: "R6"
- board text added: "R7"
- board text added: "R8"
