File: PEP003-V1-redna_i_paralelna_otpornost/PEP003-V1-redna_i_paralelna_otpornost.kicad_sch (KiCad schematic)
At the start: 23 parts, among them J1 Screw_Terminal_01x02

Commit message: PEP003 final commit, ready for production.
Parts:
- D1, D2: LCSC (none) -> C2286
- R1, R6: LCSC (none) -> C17887
- R2, R3, R5, R8: LCSC (none) -> C17936
- R4, R7: LCSC (none) -> C175514
Other:
- title: Redna i paralelna otpornost -> (none)
- moved on the sheet: H1, H2, H3, H4

Commit message: Update 1,2,3,4,5,7, lib.
Changed lines of the file:
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@@
 (kicad_sch
-	(version 20231120)
+	(version 20250114)
 	(generator "eeschema")
-	(generator_version "8.0")
+	(generator_version "9.0")
 	(paper "A4")
+	(rectangle
+		(start 172.72 12.7)
+		(end 284.48 134.62)
+		(stroke
+			(width 0)
+			(type default)
+		)
+		(fill
+			(type none)
+		)
+	)
+	(rectangle
+		(start 12.7 134.62)
+		(end 154.94 198.12)
+		(stroke
+			(width 0)
+			(type default)
+		)
+		(fill
+			(type none)
+		)
+	)
+	(rectangle
+		(start 12.7 12.7)
+		(end 96.52 134.62)
+		(stroke
+			(width 0)
+			(type default)
+		)
+		(fill
+			(type none)
+		)
+	)
+	(rectangle
+		(start 96.52 12.7)
+		(end 172.72 134.62)
+		(stroke
+			(width 0)
+			(type default)
+		)
+		(fill
+			(type none)
+		)
+	)
+	(text "Rupe za montiranje"
+		(exclude_from_sim no)
+		(at 38.354 142.494 0)
+		(effects
+			(font
+				(size 2.54 2.54)
+			)
+		)
+	)
+	(text "Paralelna otpornost\n"
+		(exclude_from_sim no)
+		(at 185.674 21.336 0)
+		(effects
+			(font
+				(size 2.54 2.54)
+			)
+			(justify left bottom)
+		)
+	)
+	(text "Redna otpornost\n"
+		(exclude_from_sim no)
+		(at 112.014 19.812 0)
+		(effects
+			(font
+				(size 2.54 2.54)
+			)
+			(justify left bottom)
+		)
+	)
+	(text "Konektor za napajanje"
+		(exclude_from_sim no)
+		(at 18.034 21.082 0)
+		(effects
+			(font
+				(size 2.54 2.54)
+			)
+			(justify left bottom)
+		)
+	)
 	(junction
 		(at 130.81 90.17)
@@
 			(width 0)
 			(type default)
-		)
-	)
-	(rectangle
-		(start 172.72 12.7)
-		(end 284.48 134.62)
-		(stroke
-			(width 0)
-			(type default)
-		)
-		(fill
-			(type none)
-		)
-	)
-	(rectangle
-		(start 12.7 134.62)
-		(end 154.94 198.12)
-		(stroke
-			(width 0)
-			(type default)
-		)
-		(fill
-			(type none)
-		)
-	)
-	(rectangle
-		(start 12.7 12.7)
-		(end 96.52 134.62)
-		(stroke
-			(width 0)
-			(type default)
-		)
-		(fill
-			(type none)
-		)
-	)
-	(rectangle
-		(start 96.52 12.7)
-		(end 172.72 134.62)
-		(stroke
-			(width 0)
-			(type default)
-		)
-		(fill
-			(type none)
-		)
-	)
-	(text "Rupe za montiranje"
-		(exclude_from_sim no)
-		(at 38.354 142.494 0)
-		(effects
-			(font
-				(size 2.54 2.54)
-			)
-		)
-	)
-	(text "Paralelna otpornost\n"
-		(exclude_from_sim no)
-		(at 185.674 21.336 0)
-		(effects
-			(font
-				(size 2.54 2.54)
-			)
-			(justify left bottom)
-		)
-	)
-	(text "Redna otpornost\n"
-		(exclude_from_sim no)
-		(at 112.014 19.812 0)
-		(effects
-			(font
-				(size 2.54 2.54)
-			)
-			(justify left bottom)
-		)
-	)
-	(text "Konektor za napajanje"
-		(exclude_from_sim no)
-		(at 18.034 21.082 0)
-		(effects
-			(font
-				(size 2.54 2.54)
-			)
-			(justify left bottom)
 		)
 	)
@@
 			)
 		)
-		(property "Description" ""
+		(property "Description" "Resistor"
 			(at 130.81 66.04 0)
 			(effects
@@
 			)
 		)
-		(property "Description" ""
+		(property "Description" "Mounting Hole without connection"
 			(at 45.72 179.07 0)
 			(effects
@@
 			)
 		)
-		(property "Description" ""
+		(property "Description" "Resistor"
 			(at 130.81 49.53 0)
 			(effects
@@
 			)
 		)
-		(property "Datasheet" "~"
+		(property "Datasheet" "https://ngspice.sourceforge.io/docs/ngspice-html-manual/manual.xhtml#subsec_Circuit_elements__device"
 			(at 222.25 109.22 0)
 			(effects
@@
 			)
 		)
-		(property "Description" ""
+		(property "Description" "0V reference potential for simulation"
 			(at 222.25 109.22 0)
 			(effects
@@
 			)
 		)
-		(property "Description" ""
+		(property "Description" "Resistor"
 			(at 257.81 82.55 0)
 			(effects
@@
 			)
 		)
-		(property "Datasheet" "~"
+		(property "Datasheet" "https://ngspice.sourceforge.io/docs/ngspice-html-manual/manual.xhtml#subsec_Circuit_elements__device"
 			(at 49.53 67.31 0)
 			(effects
@@
 			)
 		)
-		(property "Description" ""
+		(property "Description" "0V reference potential for simulation"
 			(at 49.53 67.31 0)
 			(effects
@@
 			)
 		)
-		(property "Description" ""
+		(property "Description" "Resistor"
 			(at 234.95 82.55 0)
 			(effects
@@
 			)
 		)
-		(property "Description" ""
+		(property "Description" "Jumper, 2-pole, closed/bridged"
 			(at 209.55 66.04 0)
 			(effects
@@
 			)
 		)
-		(property "Description" ""
+		(property "Description" "Jumper, 2-pole, closed/bridged"
 			(at 146.05 49.53 0)
 			(effects
@@
 			)
 		)
-		(property "Description" ""
+		(property "Description" "Resistor"
 			(at 209.55 81.28 0)
 			(effects
@@
 			)
 		)
-		(property "Description" ""
+		(property "Description" "Jumper, 2-pole, closed/bridged"
 			(at 146.05 99.06 0)
 			(effects
@@
 			)
 		)
-		(property "Datasheet" "~"
+		(property "Datasheet" "https://ngspice.sourceforge.io/docs/ngspice-html-manual/manual.xhtml#subsec_Circuit_elements__device"
 			(at 138.43 127 0)
 			(effects
@@
 			)
 		)
-		(property "Description" ""
+		(property "Description" "0V reference potential for simulation"
 			(at 138.43 127 0)
 			(effects
@@
 			)
 		)
-		(property "Description" ""
+		(property "Description" "Mounting Hole without connection"
 			(at 64.77 171.45 0)
 			(effects
@@
 			)
 		)
-		(property "Description" ""
+		(property "Description" "Light emitting diode"
 			(at 222.25 100.33 0)
 			(effects
@@
 		(property "LCSC" "C2286"
 			(at 222.25 100.33 90)
+			(effects
+				(font
+					(size 1.27 1.27)
+				)
+				(hide yes)
+			)
+		)
+		(property "Sim.Pins" "1=K 2=A"
+			(at 222.25 100.33 0)
 			(effects
 				(font
@@
 			)
 		)
-		(property "Description" ""
+		(property "Description" "Mounting Hole without connection"
 			(at 45.72 171.45 0)
 			(effects
@@
 			)
 		)
-		(property "Description" ""
+		(property "Description" "Generic screw terminal, single row, 01x02, script generated (kicad-library-utils/schlib/autogen/connector/)"
 			(at 58.42 60.96 0)
 			(effects
@@
 			)
 		)
-		(property "Description" ""
+		(property "Description" "Mounting Hole without connection"
 			(at 64.77 179.07 0)
 			(effects
@@
 			)
 		)
-		(property "Description" ""
+		(property "Description" "Resistor"
 			(at 130.81 99.06 0)
 			(effects
@@
 			)
 		)
-		(property "Description" ""
+		(property "Description" "Jumper, 2-pole, closed/bridged"
 			(at 146.05 66.04 0)
 			(effects
@@
 			)
 		)
-		(property "Description" ""
+		(property "Description" "Resistor"
 			(at 130.81 81.28 0)
 			(effects
@@
 			)
 		)
-		(property "Description" ""
+		(property "Description" "Jumper, 2-pole, closed/bridged"
 			(at 189.23 66.04 0)
 			(effects
@@
 			)
 		)
-		(property "Description" ""
+		(property "Description" "Jumper, 2-pole, closed/bridged"
 			(at 146.05 81.28 0)
 			(effects
@@
 			)
 		)
-		(property "Description" ""
+		(property "Description" "Resistor"
 			(at 189.23 81.28 0)
 			(effects
@@
 			)
 		)
-		(property "Description" ""
+		(property "Description" "Light emitting diode"
 			(at 138.43 116.84 0)
 			(effects
@@
 		(property "LCSC" "C2286"
 			(at 138.43 116.84 90)
+			(effects
+				(font
+					(size 1.27 1.27)
+				)
+				(hide yes)
+			)
+		)
+		(property "Sim.Pins" "1=K 2=A"
+			(at 138.43 116.84 0)
 			(effects
 				(font
@@
 			)
 		)
-		(property "Description" ""
+		(property "Description" "Jumper, 2-pole, closed/bridged"
 			(at 234.95 67.31 0)
 			(effects
@@
 			)
 		)
-		(property "Description" ""
+		(property "Description" "Jumper, 2-pole, closed/bridged"
 			(at 257.81 67.31 0)
 			(effects
@@
 		)
 	)
+	(embedded_fonts no)
 )
