File: PEP005-V1-dzulov_zakon/PEP005-V1-dzulov_zakon.kicad_pcb (KiCad board)
At the start: 2 copper layers, 45 x 45 mm, 11 parts, among them J1 Conn_01x01_Socket, J2 Screw_Terminal_01x02, J3 Conn_01x01_Socket

Commit message: PEP005 final.
Parts:
- added G***: LOGO, logo:logo, B.Cu at (126.8, 97.2)
- added REF**: ele_petnica_logo, PEP_library:ele_petnica_logo, F.Cu at (133.5, 97.0)
- R1, R2: value 100k -> 100
- R3: value 100k -> 1k
- R4: value 100k -> 10k
Routing:
- net 0: track 7.35 -> 67.7 mm, vias 113 -> 0
- net Input voltage: track 59.5 -> 77.6 mm, vias 4 -> 0
- net (no net): vias 0 -> 109
- removed copper zone on B.Cu, net 0
Other:
- board text added: "*Light Emiting Resistor"
- board text added: "LER*"
- board text added: "PEP 005"
- board text removed: "Light emiting resistor"
- board text removed: "PEP 004"
- board text removed: "puni"

Commit message: Update 1,2,3,4,5,7, lib.
Parts:
- removed the G*** at (126.8, 97.2)
- added G***: LOGO, PEP_library:petnica_logo, F.Cu at (142.5, 75.0)
- added REF**: R_silk_symbol, PEP_library:R_silk_symbol, F.Cu at (127.0, 68.1)
- J2: footprint TerminalBlock_Phoenix:TerminalBlock_Phoenix_MKDS-1,5-2-5.08_1x02_P5.08mm_Horizontal -> PEP_library:TerminalBlock_Phoenix_MKDS-1,5-2-5.08_1x02_P5.08mm_Horizontal
- R1, R2, R3, R4: footprint Resistor_SMD:R_1206_3216Metric_Pad1.30x1.75mm_HandSolder -> PEP_library:R_smd_1206
- moved J1 28.7 mm to (127.5, 66.5)
- moved R2 19.9 mm to (131.9, 80.0), turned to 0 degrees
- moved J2 16.9 mm to (114.3, 78.0), turned to -90 degrees
- moved J3 16.3 mm to (136.5, 66.5)
- moved R1 14.8 mm to (131.9, 73.5), turned to 0 degrees
- moved REF** 12.1 mm to (143.0, 89.5)
- moved R4 8.09 mm to (131.9, 93.0), turned to 0 degrees
- moved R3 2.01 mm to (131.9, 86.5), turned to 0 degrees
Routing:
- net Input voltage: track 77.6 -> 45.7 mm
- net 0: track 67.7 -> 62.2 mm
- removed copper zone on F.Cu, net 0
- removed copper zone on F.Cu, net Input voltage
Other:
- board text added: "*Light emiting resistor"
- board text added: "LER"
- board text added: "R1"
- board text added: "R2"
- board text added: "R3"
- board text added: "R4"
- board text removed: "*Light Emiting Resistor"
- board text removed: "LER*"
