File: PEP005-V1-dzulov_zakon/PEP005-V1-dzulov_zakon.kicad_sch (KiCad schematic)
At the start: 12 parts, among them J1 Conn_01x01_Socket, J2 Screw_Terminal_01x02, J3 Conn_01x01_Socket

Commit message: PEP005 final.
Parts:
- J2: LCSC Part Number (none) -> C3018698
- R1, R2: value 100k -> 100; JLCPCB Footprint (none) -> 1206; LCSC Part Number (none) -> C17900
- R3: value 100k -> 1k; JLCPCB Footprint (none) -> 1206; LCSC Part Number (none) -> C17900
- R4: value 100k -> 10k; JLCPCB Footprint (none) -> 1206; LCSC Part Number (none) -> C17900
Changed lines of the file:
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@@
 (kicad_sch
-	(version 20231120)
+	(version 20250114)
 	(generator "eeschema")
-	(generator_version "8.0")
+	(generator_version "9.0")
 	(paper "A5")
 	(title_block
@@
 		(rev "v1")
 	)
+	(rectangle
+		(start 12.065 12.065)
+		(end 69.85 104.14)
+		(stroke
+			(width 0)
+			(type default)
+		)
+		(fill
+			(type none)
+		)
+	)
+	(rectangle
+		(start 12.065 104.14)
+		(end 83.82 135.89)
+		(stroke
+			(width 0)
+			(type default)
+		)
+		(fill
+			(type none)
+		)
+	)
+	(rectangle
+		(start 69.85 12.065)
+		(end 192.405 104.14)
+		(stroke
+			(width 0)
+			(type default)
+		)
+		(fill
+			(type none)
+		)
+	)
+	(text "zamneljivi i zapaljiv otpornik\n"
+		(exclude_from_sim no)
+		(at 156.21 54.864 90)
+		(effects
+			(font
+				(size 2.54 2.54)
+			)
+		)
+	)
+	(text "Rupe za montiranje\n"
+		(exclude_from_sim no)
+		(at 17.78 109.22 0)
+		(effects
+			(font
+				(size 2.54 2.54)
+			)
+			(justify left bottom)
+		)
+	)
+	(text "otpornik okružen bakrom\n"
+		(exclude_from_sim no)
+		(at 77.216 61.468 90)
+		(effects
+			(font
+				(size 2.54 2.54)
+			)
+		)
+	)
+	(text "Konektor za napajanje"
+		(exclude_from_sim no)
+		(at 12.7 17.78 0)
+		(effects
+			(font
+				(size 2.54 2.54)
+			)
+			(justify left bottom)
+		)
+	)
+	(text "Otpornici sa gradijentom disipacije\n"
+		(exclude_from_sim no)
+		(at 71.12 17.78 0)
+		(effects
+			(font
+				(size 2.54 2.54)
+			)
+			(justify left bottom)
+		)
+	)
 	(junction
 		(at 114.3 30.48)
@@
 			(width 0)
 			(type default)
-		)
-	)
-	(rectangle
-		(start 12.065 12.065)
-		(end 69.85 104.14)
-		(stroke
-			(width 0)
-			(type default)
-		)
-		(fill
-			(type none)
-		)
-	)
-	(rectangle
-		(start 12.065 104.14)
-		(end 83.82 135.89)
-		(stroke
-			(width 0)
-			(type default)
-		)
-		(fill
-			(type none)
-		)
-	)
-	(rectangle
-		(start 69.85 12.065)
-		(end 192.405 104.14)
-		(stroke
-			(width 0)
-			(type default)
-		)
-		(fill
-			(type none)
-		)
-	)
-	(text "zamneljivi i zapaljiv otpornik\n"
-		(exclude_from_sim no)
-		(at 156.21 54.864 90)
-		(effects
-			(font
-				(size 2.54 2.54)
-			)
-		)
-	)
-	(text "Rupe za montiranje\n"
-		(exclude_from_sim no)
-		(at 17.78 109.22 0)
-		(effects
-			(font
-				(size 2.54 2.54)
-			)
-			(justify left bottom)
-		)
-	)
-	(text "otpornik okružen bakrom\n"
-		(exclude_from_sim no)
-		(at 77.216 61.468 90)
-		(effects
-			(font
-				(size 2.54 2.54)
-			)
-		)
-	)
-	(text "Konektor za napajanje"
-		(exclude_from_sim no)
-		(at 12.7 17.78 0)
-		(effects
-			(font
-				(size 2.54 2.54)
-			)
-			(justify left bottom)
-		)
-	)
-	(text "Otpornici sa gradijentom disipacije\n"
-		(exclude_from_sim no)
-		(at 71.12 17.78 0)
-		(effects
-			(font
-				(size 2.54 2.54)
-			)
-			(justify left bottom)
 		)
 	)
@@
 			)
 		)
-		(property "Value" "100k"
+		(property "Value" "100"
 			(at 84.328 58.928 0)
 			(effects
@@
 			)
 		)
-		(property "Datasheet" "~"
+		(property "Datasheet" "https://jlcpcb.com/api/file/downloadByFileSystemAccessId/8579705871070658560"
 			(at 90.17 58.42 0)
 			(effects
@@
 			)
 		)
+		(property "LCSC Part Number" "C17900"
+			(at 90.17 58.42 0)
+			(effects
+				(font
+					(size 1.27 1.27)
+				)
+				(hide yes)
+			)
+		)
+		(property "JLCPCB Footprint" "1206"
+			(at 90.17 58.42 0)
+			(effects
+				(font
+					(size 1.27 1.27)
+				)
+				(hide yes)
+			)
+		)
 		(pin "1"
 		)
@@
 			)
 		)
-		(property "Datasheet" "~"
+		(property "Datasheet" "https://wmsc.lcsc.com/wmsc/upload/file/pdf/v2/lcsc/2301061230_DORABO-DB127V-5-08-2P-GN-S_C3018698.pdf"
 			(at 48.26 53.34 0)
 			(effects
@@
 			)
 		)
+		(property "LCSC Part Number" "C3018698"
+			(at 48.26 53.34 0)
+			(effects
+				(font
+					(size 1.27 1.27)
+				)
+				(hide yes)
+			)
+		)
 		(pin "1"
 		)
@@
 			)
 		)
-		(property "Value" "100k"
+		(property "Value" "10k"
 			(at 119.888 58.928 0)
 			(effects
@@
 			)
 		)
-		(property "Datasheet" "~"
+		(property "Datasheet" "https://jlcpcb.com/api/file/downloadByFileSystemAccessId/8579705871070658560"
 			(at 125.73 58.42 0)
 			(effects
@@
 		)
 		(property "Description" ""
+			(at 125.73 58.42 0)
+			(effects
+				(font
+					(size 1.27 1.27)
+				)
+				(hide yes)
+			)
+		)
+		(property "LCSC Part Number" "C17900"
+			(at 125.73 58.42 0)
+			(effects
+				(font
+					(size 1.27 1.27)
+				)
+				(hide yes)
+			)
+		)
+		(property "JLCPCB Footprint" "1206"
 			(at 125.73 58.42 0)
 			(effects
@@
 			)
 		)
-		(property "Value" "100k"
+		(property "Value" "1k"
 			(at 108.458 58.928 0)
 			(effects
@@
 			)
 		)
-		(property "Datasheet" "~"
+		(property "Datasheet" "https://jlcpcb.com/api/file/downloadByFileSystemAccessId/8579705871070658560"
 			(at 114.3 58.42 0)
 			(effects
@@
 		)
 		(property "Description" ""
+			(at 114.3 58.42 0)
+			(effects
+				(font
+					(size 1.27 1.27)
+				)
+				(hide yes)
+			)
+		)
+		(property "LCSC Part Number" "C17900"
+			(at 114.3 58.42 0)
+			(effects
+				(font
+					(size 1.27 1.27)
+				)
+				(hide yes)
+			)
+		)
+		(property "JLCPCB Footprint" "1206"
 			(at 114.3 58.42 0)
 			(effects
@@
 			)
 		)
-		(property "Value" "100k"
+		(property "Value" "100"
 			(at 97.028 58.928 0)
 			(effects
@@
 			)
 		)
-		(property "Datasheet" "~"
+		(property "Datasheet" "https://jlcpcb.com/api/file/downloadByFileSystemAccessId/8579705871070658560"
 			(at 102.87 58.42 0)
 			(effects
@@
 		)
 		(property "Description" ""
+			(at 102.87 58.42 0)
+			(effects
+				(font
+					(size 1.27 1.27)
+				)
+				(hide yes)
+			)
+		)
+		(property "LCSC Part Number" "C17900"
+			(at 102.87 58.42 0)
+			(effects
+				(font
+					(size 1.27 1.27)
+				)
+				(hide yes)
+			)
+		)
+		(property "JLCPCB Footprint" "1206"
 			(at 102.87 58.42 0)
 			(effects
@@
 		)
 	)
+	(embedded_fonts no)
 )

Commit message: Update 1,2,3,4,5,7, lib.
Parts:
- J2: footprint TerminalBlock_Phoenix:TerminalBlock_Phoenix_MKDS-1,5-2-5.08_1x02_P5.08mm_Horizontal -> PEP_library:TerminalBlock_Phoenix_MKDS-1,5-2-5.08_1x02_P5.08mm_Horizontal
- R1, R2, R3, R4: footprint Resistor_SMD:R_1206_3216Metric_Pad1.30x1.75mm_HandSolder -> PEP_library:R_smd_1206
Changed lines of the file:
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@@
 			)
 		)
-		(property "Footprint" "Resistor_SMD:R_1206_3216Metric_Pad1.30x1.75mm_HandSolder"
+		(property "Footprint" "PEP_library:R_smd_1206"
 			(at 88.392 58.42 90)
 			(effects
@@
 			)
 		)
-		(property "Footprint" "TerminalBlock_Phoenix:TerminalBlock_Phoenix_MKDS-1,5-2-5.08_1x02_P5.08mm_Horizontal"
+		(property "Footprint" "PEP_library:TerminalBlock_Phoenix_MKDS-1,5-2-5.08_1x02_P5.08mm_Horizontal"
 			(at 48.26 53.34 0)
 			(effects
@@
 			)
 		)
-		(property "Datasheet" "https://wmsc.lcsc.com/wmsc/upload/file/pdf/v2/lcsc/2301061230_DORABO-DB127V-5-08-2P-GN-S_C3018698.pdf"
+		(property "Datasheet" "~"
 			(at 48.26 53.34 0)
 			(effects
@@
 			)
 		)
-		(property "Description" ""
+		(property "Description" "Generic screw terminal, single row, 01x02, script generated (kicad-library-utils/schlib/autogen/connector/)"
 			(at 48.26 53.34 0)
 			(effects
@@
 			)
 		)
-		(property "Footprint" "Resistor_SMD:R_1206_3216Metric_Pad1.30x1.75mm_HandSolder"
+		(property "Footprint" "PEP_library:R_smd_1206"
 			(at 123.952 58.42 90)
 			(effects
@@
 			)
 		)
-		(property "Footprint" "Resistor_SMD:R_1206_3216Metric_Pad1.30x1.75mm_HandSolder"
+		(property "Footprint" "PEP_library:R_smd_1206"
 			(at 112.522 58.42 90)
 			(effects
@@
 			)
 		)
-		(property "Footprint" "Resistor_SMD:R_1206_3216Metric_Pad1.30x1.75mm_HandSolder"
+		(property "Footprint" "PEP_library:R_smd_1206"
 			(at 101.092 58.42 90)
 			(effects
