File: PEP009-V1-LC_rezonantno_kolo/PEP009-V1-LC_rezonantno_kolo.kicad_pcb (KiCad board)
At the start: 2 copper layers, 45 x 45 mm, 21 parts, among them J1 Screw_Terminal_01x02, J2 Conn_01x01_Pin, J3 Conn_01x01_Pin, J4 Conn_01x01_Pin

Commit message: PEP009 final commit, ready for production.
Parts:
- moved REF** 3.49 mm to (152.7, 74.5)
Changed lines of the file:
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@@
 	(footprint "PEP_library:ele_petnica_logo"
 		(layer "F.Cu")
-		(at 149.325 73.7)
+		(at 152.725 74.476394)
 		(property "Reference" "REF**"
 			(at 0.25 -5.5 0)

Commit message: Klema i kondenzatori zamenjeni sa onima iz PEP biblioteke. Naziv i broj plocice izmenjeni po standardnim pravilima
Parts:
- added H1: MountingHole, MountingHole:MountingHole_3.2mm_M3_ISO14580_Pad_TopBottom, F.Cu at (3.02, 3.02)
- added H2: MountingHole, MountingHole:MountingHole_3.2mm_M3_ISO14580_Pad_TopBottom, F.Cu at (3.02, 10.1)
- added H3: MountingHole, MountingHole:MountingHole_3.2mm_M3_ISO14580_Pad_TopBottom, F.Cu at (3.02, 17.1)
- added H4: MountingHole, MountingHole:MountingHole_3.2mm_M3_ISO14580_Pad_TopBottom, F.Cu at (3.02, 24.2)
- C1, C2, C3: footprint Capacitor_SMD:C_1206_3216Metric -> PEP_library:C_1206_3216Metric
- J1: footprint TerminalBlock_Phoenix:TerminalBlock_Phoenix_MKDS-1,5-2-5.08_1x02_P5.08mm_Horizontal -> PEP_library:TerminalBlock_Phoenix_MKDS-1,5-2-5.08_1x02_P5.08mm_Horizontal
- R1: footprint Resistor_SMD:R_1206_3216Metric -> PEP_library:R_smd
Connections:
- J1 pad 2: GND -> 0
Other:
- board text removed: "+"
- board text removed: "-"
- board text removed: "V_{in}"
